File: CDiGenesis.kicad_sch (KiCad schematic)
At the start: 4 parts, among them J1 Genesis, J2 CDi, U1 ATtiny1616-M

Commit message: Effectively finalise PCB design
Parts:
- added H1, H2: M2, MountingHole:MountingHole_2.2mm_M2, symbol Mechanical:MountingHole
- added J3: Conn_01x03, UPDI:UPDI Pads, symbol Connector_Generic:Conn_01x03
Connections:
- net +5V: now also J3.1 (Pin_1)
- net BTN_A/B: now also U1.7 (PA6); no longer U1.6 (PA5)
- net BTN_S/C: now also U1.20 (PA1); no longer U1.7 (PA6)
- net D_Down: now also U1.6 (PA5); no longer U1.1 (PA2)
- net D_Right: now also U1.1 (PA2); no longer U1.5 (PA4)
- net D_Up: now also U1.8 (PA7); no longer U1.20 (PA1)
- net GND: now also J3.3 (Pin_3)
- net RTS: now also U1.15 (PC0); no longer U1.10 (PB4)
- net Select: now also U1.5 (PA4); no longer U1.8 (PA7)
- net UPDI: now reaches U1.19 (~{RESET}/PA0)
- net UPDI: now also J3.2 (Pin_2)

Commit message: Fix connector type
Parts:
- removed J1: Genesis, Connector_Dsub:DSUB-9_Socket_Horizontal_P2.77x2.84mm_EdgePinOffset4.94mm_Housed_MountingHolesOffset4.94mm, symbol Connector:DE9_Socket_MountingHoles
- added J1: Genesis, Connector_Dsub:DSUB-9_Pins_Horizontal_P2.77x2.84mm_EdgePinOffset4.94mm_Housed_MountingHolesOffset4.94mm, symbol Connector:DE9_Pins_MountingHoles
Connections:
- net +5V: now also J1.5
- net BTN_A/B: now also U1.1 (PA2), J1.6; no longer U1.7 (PA6)
- net BTN_S/C: now also U1.8 (PA7), J1.9; no longer U1.20 (PA1)
- net D_Down: now also U1.2 (PA3), J1.2; no longer U1.6 (PA5)
- net D_Left: now also U1.5 (PA4), J1.3; no longer U1.2 (PA3)
- net D_Right: now also U1.7 (PA6), J1.4; no longer U1.1 (PA2)
- net D_Up: now also U1.20 (PA1), J1.1; no longer U1.8 (PA7)
- net GND: now also J1.0 (PAD), J1.8
- net Select: now also U1.6 (PA5), J1.7; no longer U1.5 (PA4)
