File: KiCad/CDiGenesis.kicad_sch (KiCad schematic)
At the start: 7 parts, among them J1 Genesis, J2 CDi, J3 Conn_01x03, U1 ATtiny1616-M

Commit message: Add silkscreen, nearing code completion
Connections:
- net BTN_A/B renamed BTN_B/A
- net BTN_S/C renamed BTN_C/S
Changed lines of the file:
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@@
 		)
 	)
-	(label "BTN_A{slash}B"
+	(label "BTN_B{slash}A"
 		(at 90.17 74.93 180)
 		(effects
@@
 		)
 	)
-	(label "BTN_A{slash}B"
+	(label "BTN_B{slash}A"
 		(at 172.72 97.79 0)
 		(effects
@@
 		)
 	)
-	(label "BTN_S{slash}C"
+	(label "BTN_C{slash}S"
 		(at 172.72 82.55 0)
 		(effects
@@
 		)
 	)
-	(label "BTN_S{slash}C"
+	(label "BTN_C{slash}S"
 		(at 90.17 87.63 180)
 		(effects

Commit message: Effectively finalise code, remove SELECT nonsense
Connections:
- net +5V: no longer J1.5
- net D_Right: now also U1.6 (PA5); no longer U1.7 (PA6)
- net BTN_B/A renamed BTN_B
- net BTN_C/S: no longer names the net of U1.8 (PA7)
- net BTN_C/S: no longer J1.9
- net Select: no longer names the net of J1.7
- net Select: no longer U1.6 (PA5)
- new net BTN_C: J1.9, U1.7 (PA6)
- no-connect marks 12 -> 15

Commit message: Revert PCB changes, will modify code
This reverts commit 0f8f6d9ed579b1546b77e135067905f4b0f0e6bf.
Connections:
- net +5V: now also J1.5
- net D_Right: now also U1.7 (PA6); no longer U1.6 (PA5)
- net Select: now reaches J1.7
- net Select: now also U1.6 (PA5)
- net BTN_C/S: now reaches U1.8 (PA7)
- net BTN_C/S: now also J1.9
- net BTN_B renamed BTN_B/A
- removed net BTN_C: J1.9, U1.7 (PA6)
- no-connect marks 15 -> 12
